Commit message: Bugfixing

File: test.urdf (robot description, URDF)
Before this commit: robot lbr_iiwa, 5 links, 4 joints
Links:
- link link3: mass 5 -> 1
Joints:
- joint joint1: limit lower=-3.14159265359 upper=3.14159265359 effort=5 velocity=200 -> lower=-3.14159265359 upper=3.14159265359 effort=500 velocity=200
- joint joint2: limit lower=-3.14159265359 upper=3.14159265359 effort=5 velocity=200 -> lower=-3.14159265359 upper=3.14159265359 effort=500 velocity=200
- joint joint3: limit lower=-3.14159265359 upper=3.14159265359 effort=500 velocity=200 -> lower=-3.14159265359 upper=3.14159265359 effort=100 velocity=200; type fixed -> revolute

Commit message: Dynamic path planner integrated

File: test.urdf (robot description, URDF)
Before this commit: robot lbr_iiwa, 5 links, 4 joints
Joints:
- joint joint1: limit lower=-3.14159265359 upper=3.14159265359 effort=500 velocity=200 -> lower=-3.14159265359 upper=3.14159265359 effort=400 velocity=200
- joint joint2: limit lower=-3.14159265359 upper=3.14159265359 effort=500 velocity=200 -> lower=-3.14159265359 upper=3.14159265359 effort=400 velocity=200
- joint joint3: limit lower=-3.14159265359 upper=3.14159265359 effort=100 velocity=200 -> lower=-3.14159265359 upper=3.14159265359 effort=400 velocity=200

Commit message: Included nonlinear propagator for simulation interface

File: test.urdf (robot description, URDF)
Before this commit: robot lbr_iiwa, 5 links, 4 joints
Joints:
- joint joint1: limit lower=-3.14159265359 upper=3.14159265359 effort=400 velocity=200 -> lower=-3.14159265359 upper=3.14159265359 effort=500 velocity=200
- joint joint2: limit lower=-3.14159265359 upper=3.14159265359 effort=400 velocity=200 -> lower=-3.14159265359 upper=3.14159265359 effort=200 velocity=200
- joint joint3: limit lower=-3.14159265359 upper=3.14159265359 effort=400 velocity=200 -> lower=-3.14159265359 upper=3.14159265359 effort=200 velocity=200

Commit message: Fully integrated dynamic path planner

File: test.urdf (robot description, URDF)
Before this commit: robot lbr_iiwa, 5 links, 4 joints
Links:
- link end_effector: mass None -> 0.0000001

Commit message: Parameter fixing

File: test.urdf (robot description, URDF)
Before this commit: robot lbr_iiwa, 5 links, 4 joints
Joints:
- joint joint4: limit lower=-3.14159265359 upper=3.14159265359 effort=10 velocity=10 -> lower=-3.14159265359 upper=3.14159265359 effort=200 velocity=10

Commit message: Make goal area a tiny bit smaller than the nominal goal area in order to account for errors

File: test.urdf (robot description, URDF)
Before this commit: robot lbr_iiwa, 5 links, 4 joints
Joints:
- joint joint4: limit lower=-3.14159265359 upper=3.14159265359 effort=200 velocity=10 -> lower=-3.14159265359 upper=3.14159265359 effort=200 velocity=0

Commit message: Parameter tuning

File: test.urdf (robot description, URDF)
Before this commit: robot lbr_iiwa, 5 links, 4 joints
Joints:
- joint joint4: limit lower=-3.14159265359 upper=3.14159265359 effort=200 velocity=0 -> lower=-3.14159265359 upper=3.14159265359 effort=200 velocity=1

Commit message: Linearize about arbitrary state or closest steady state (optional)

File: test.urdf (robot description, URDF)
Before this commit: robot lbr_iiwa, 5 links, 4 joints
Links:
- removed link link3
- link end_effector: mass 0.0000001 -> None
Joints:
- removed joint joint4
- joint joint3: child link3 -> end_effector; type revolute -> fixed

Commit message: Cleanup and bugfixing

File: test.urdf (robot description, URDF)
Before this commit: robot lbr_iiwa, 4 links, 3 joints
Links:
- added link link3, mass 1; collision box size=1 0.15 0.15; visual box size=1 0.15 0.15
Joints:
- added joint joint4: type fixed, parent link3, child end_effector, origin xyz=1 0 0 rpy=0 0 0, axis 0 0 1, limit lower=-3.14159265359 upper=3.14159265359 effort=200 velocity=1
- joint joint3: child end_effector -> link3; type fixed -> revolute

Commit message: Testing

File: test.urdf (robot description, URDF)
Before this commit: robot lbr_iiwa, 5 links, 4 joints
Links:
- link link1: mass 1 -> 0.5
- link link2: mass 1 -> 0.5
- link link3: mass 1 -> 0.5
Joints:
- joint joint1: limit lower=-3.14159265359 upper=3.14159265359 effort=500 velocity=200 -> lower=-3.14159265359 upper=3.14159265359 effort=300 velocity=200
- joint joint2: limit lower=-3.14159265359 upper=3.14159265359 effort=200 velocity=200 -> lower=-3.14159265359 upper=3.14159265359 effort=100 velocity=200
- joint joint3: limit lower=-3.14159265359 upper=3.14159265359 effort=200 velocity=200 -> lower=-3.14159265359 upper=3.14159265359 effort=100 velocity=200

Commit message: testing

File: test.urdf (robot description, URDF)
Before this commit: robot lbr_iiwa, 5 links, 4 joints
Joints:
- joint joint1: limit lower=-3.14159265359 upper=3.14159265359 effort=300 velocity=200 -> lower=-3.14159265359 upper=3.14159265359 effort=40 velocity=200
- joint joint2: limit lower=-3.14159265359 upper=3.14159265359 effort=100 velocity=200 -> lower=-3.14159265359 upper=3.14159265359 effort=10 velocity=200
- joint joint3: limit lower=-3.14159265359 upper=3.14159265359 effort=100 velocity=200 -> lower=-3.14159265359 upper=3.14159265359 effort=10 velocity=200
- joint joint4: limit lower=-3.14159265359 upper=3.14159265359 effort=200 velocity=1 -> lower=-3.14159265359 upper=3.14159265359 effort=20 velocity=1

Commit message: Testing

File: test.urdf (robot description, URDF)
Before this commit: robot lbr_iiwa, 5 links, 4 joints
Links:
- link link1: mass 0.5 -> 1
- link link2: mass 0.5 -> 1
- link link3: mass 0.5 -> 1

Commit message: Replaced physics engine in propagator with Bulirsch-Stoer integration

File: test.urdf (robot description, URDF)
Before this commit: robot lbr_iiwa, 5 links, 4 joints
Joints:
- joint joint1: limit lower=-3.14159265359 upper=3.14159265359 effort=40 velocity=200 -> lower=-3.1 upper=3.1 effort=50 velocity=10
- joint joint2: limit lower=-3.14159265359 upper=3.14159265359 effort=10 velocity=200 -> lower=-3.1 upper=3.1 effort=30 velocity=10
- joint joint3: limit lower=-3.14159265359 upper=3.14159265359 effort=10 velocity=200 -> lower=-3.1 upper=3.1 effort=20 velocity=10
- joint joint4: limit lower=-3.14159265359 upper=3.14159265359 effort=20 velocity=1 -> lower=-3.1 upper=3.1 effort=20 velocity=1

Commit message: testing

File: test.urdf (robot description, URDF)
Before this commit: robot lbr_iiwa, 5 links, 4 joints
Joints:
- joint joint1: limit lower=-3.1 upper=3.1 effort=50 velocity=10 -> lower=-3.1 upper=3.1 effort=50 velocity=15
- joint joint2: limit lower=-3.1 upper=3.1 effort=30 velocity=10 -> lower=-3.1 upper=3.1 effort=20 velocity=15
- joint joint3: limit lower=-3.1 upper=3.1 effort=20 velocity=10 -> lower=-3.1 upper=3.1 effort=15 velocity=15

Commit message: Bugfixing

File: test.urdf (robot description, URDF)
Before this commit: robot lbr_iiwa, 5 links, 4 joints
Joints:
- joint joint1: limit lower=-3.1 upper=3.1 effort=50 velocity=15 -> lower=-3.1 upper=3.1 effort=30 velocity=15
- joint joint3: limit lower=-3.1 upper=3.1 effort=15 velocity=15 -> lower=-3.1 upper=3.1 effort=5 velocity=15

Commit message: Testing

File: test.urdf (robot description, URDF)
Before this commit: robot lbr_iiwa, 5 links, 4 joints
Joints:
- joint joint1: limit lower=-3.1 upper=3.1 effort=30 velocity=15 -> lower=-3.1 upper=3.1 effort=50 velocity=15
- joint joint3: limit lower=-3.1 upper=3.1 effort=5 velocity=15 -> lower=-3.1 upper=3.1 effort=10 velocity=15

Commit message: Bugfixing

File: test.urdf (robot description, URDF)
Before this commit: robot lbr_iiwa, 5 links, 4 joints
Joints:
- joint joint4: axis 0 0 1 -> 0 0 0

Commit message: Use robot class instead of parametrized link dimensions

File: test.urdf (robot description, URDF)
Before this commit: robot lbr_iiwa, 5 links, 4 joints
Joints:
- joint joint2: origin xyz=1 0 0 rpy=0 0 0 -> xyz=1 0 0 rpy=-1.57079632679489661923 0 0

Commit message: ALmost done

File: test.urdf (robot description, URDF)
Before this commit: robot lbr_iiwa, 5 links, 4 joints
Joints:
- joint joint2: origin xyz=1 0 0 rpy=-1.57079632679489661923 0 0 -> xyz=1 0 0 rpy=0 0 0
