Commit message: Bugfixing

File: model/test.urdf (robot description, URDF)
Before this commit: robot lbr_iiwa, 5 links, 4 joints
Joints:
- joint joint1: limit lower=-3.1 upper=3.1 effort=50 velocity=15 -> lower=-3.1 upper=3.1 effort=200 velocity=15
- joint joint2: limit lower=-3.1 upper=3.1 effort=20 velocity=15 -> lower=-3.1 upper=3.1 effort=200 velocity=15
- joint joint3: limit lower=-3.1 upper=3.1 effort=10 velocity=15 -> lower=-3.1 upper=3.1 effort=100 velocity=15

Commit message: Bugfixing

File: model/test.urdf (robot description, URDF)
Before this commit: robot lbr_iiwa, 5 links, 4 joints
Joints:
- joint joint1: limit lower=-3.1 upper=3.1 effort=200 velocity=15 -> lower=-3.14 upper=3.14 effort=50 velocity=10
- joint joint2: limit lower=-3.1 upper=3.1 effort=200 velocity=15 -> lower=-3.14 upper=3.14 effort=50 velocity=5
- joint joint3: limit lower=-3.1 upper=3.1 effort=100 velocity=15 -> lower=-3.14 upper=3.14 effort=50 velocity=3
- joint joint4: limit lower=-3.1 upper=3.1 effort=20 velocity=1 -> lower=-3.14 upper=3.14 effort=20 velocity=1

Commit message: Fixes in model generator and goal position description

File: model/test.urdf (robot description, URDF)
Before this commit: robot lbr_iiwa, 5 links, 4 joints
Links:
- link link3: mass 1 -> 5
Joints:
- joint joint1: limit lower=-3.14 upper=3.14 effort=50 velocity=10 -> lower=-3.14159265358979323846 upper=3.14159265358979323846 effort=150 velocity=10; origin xyz=0 0 0 rpy=0 0 0 -> xyz=0 0 5 rpy=0 0 0
- joint joint2: limit lower=-3.14 upper=3.14 effort=50 velocity=5 -> lower=-3.14159265358979323846 upper=3.14159265358979323846 effort=70 velocity=10; origin xyz=1 0 0 rpy=0 0 0 -> xyz=1 0 0 rpy=-1.57079632679489661923 0 0
- joint joint3: limit lower=-3.14 upper=3.14 effort=50 velocity=3 -> lower=-3.14159265358979323846 upper=3.14159265358979323846 effort=40 velocity=10
- joint joint4: axis 0 0 0 -> 0 0 1; limit lower=-3.14 upper=3.14 effort=20 velocity=1 -> lower=-3.1 upper=3.1 effort=2 velocity=10

Commit message: Bugfixing

File: model/test.urdf (robot description, URDF)
Before this commit: robot lbr_iiwa, 5 links, 4 joints
Links:
- link end_effector: geometry collision box size=0 0 0

Commit message: Use Adams-Bashford numerical integrator. Invert inertia matrix at runtime

File: model/test.urdf (robot description, URDF)
Before this commit: robot lbr_iiwa, 5 links, 4 joints
Links:
- added link link4, mass 1; collision box size=1 0.15 0.15; visual box size=1 0.15 0.15
- link link3: mass 5 -> 1
Joints:
- added joint joint5: type fixed, parent link4, child end_effector, origin xyz=1 0 0 rpy=0 0 0, axis 0 0 1, limit lower=-3.14159265358979323846 upper=3.14159265358979323846 effort=40 velocity=10
- joint joint4: child end_effector -> link4; limit lower=-3.1 upper=3.1 effort=2 velocity=10 -> lower=-3.14159265358979323846 upper=3.14159265358979323846 effort=40 velocity=10; origin xyz=1 0 0 rpy=0 0 0 -> xyz=1 0 0 rpy=1.57079632679489661923 0 0; type fixed -> revolute

Commit message: More output

File: model/test.urdf (robot description, URDF)
Before this commit: robot lbr_iiwa, 6 links, 5 joints
Links:
- removed link link4
Joints:
- removed joint joint5
- joint joint4: child link4 -> end_effector; origin xyz=1 0 0 rpy=1.57079632679489661923 0 0 -> xyz=1 0 0 rpy=0 0 0; type revolute -> fixed

Commit message: test

File: model/test.urdf (robot description, URDF)
Before this commit: robot lbr_iiwa, 5 links, 4 joints
Links:
- added link link4, mass 1; collision box size=1 0.15 0.15; visual box size=1 0.15 0.15
Joints:
- added joint joint5: type fixed, parent link4, child end_effector, origin xyz=1 0 0 rpy=0 0 0, axis 0 0 1, limit lower=-3.14159265358979323846 upper=3.14159265358979323846 effort=40 velocity=10
- joint joint2: origin xyz=1 0 0 rpy=0 0 0 -> xyz=1 0 0 rpy=-1.57079632679489661923 0 0
- joint joint4: child end_effector -> link4; origin xyz=1 0 0 rpy=0 0 0 -> xyz=1 0 0 rpy=1.57079632679489661923 0 0; type fixed -> revolute

Commit message: test

File: model/test.urdf (robot description, URDF)
Before this commit: robot lbr_iiwa, 6 links, 5 joints
Links:
- removed link link4
Joints:
- removed joint joint5
- joint joint4: child link4 -> end_effector; type revolute -> fixed

Commit message: Bugfixing

File: model/test.urdf (robot description, URDF)
Before this commit: robot lbr_iiwa, 5 links, 4 joints
Links:
- added link link4, mass 1; collision box size=1 0.15 0.15; visual box size=1 0.15 0.15
Joints:
- added joint joint5: type fixed, parent link4, child end_effector, origin xyz=1 0 0 rpy=0 0 0, axis 0 0 1, limit lower=-3.14159265358979323846 upper=3.14159265358979323846 effort=40 velocity=10
- joint joint4: child end_effector -> link4; type fixed -> revolute
