Commit message: More output

File: model/test_3dof.urdf (robot description, URDF)
Before this commit: robot lbr_iiwa, 5 links, 4 joints
Joints:
- joint joint3: limit lower=-3.14159265358979323846 upper=3.14159265358979323846 effort=40 velocity=10 -> lower=-3.14159265358979323846 upper=3.14159265358979323846 effort=60 velocity=10
- joint joint4: origin xyz=1 0 0 rpy=0 0 0 -> xyz=1 0 0 rpy=1.57079632679489661923 0 0
