Commit message: Updated 6dof model

File: model/test_6dof.urdf (robot description, URDF)
Before this commit: robot lbr_iiwa, 8 links, 7 joints
Links:
- link link1: mass 1 -> 3.0
- link link2: mass 1 -> 2.0
- link link3: mass 1 -> 0.2
- link link4: mass 1 -> 0.2
- link link5: mass 1 -> 0.1
- link link6: mass 1 -> 0.1
Joints:
- joint joint1: limit lower=-3.14159265358979323846 upper=3.14159265358979323846 effort=180 velocity=10 -> lower=-3.14159265358979323846 upper=3.14159265358979323846 effort=20 velocity=2
- joint joint2: limit lower=-3.14159265358979323846 upper=3.14159265358979323846 effort=100 velocity=10 -> lower=-3.14159265358979323846 upper=3.14159265358979323846 effort=15 velocity=2
- joint joint3: limit lower=-3.14159265358979323846 upper=3.14159265358979323846 effort=80 velocity=10 -> lower=-3.14159265358979323846 upper=3.14159265358979323846 effort=15 velocity=2
- joint joint4: limit lower=-3.14159265358979323846 upper=3.14159265358979323846 effort=60 velocity=10 -> lower=-3.14159265358979323846 upper=3.14159265358979323846 effort=10 velocity=2
- joint joint5: limit lower=-3.14159265358979323846 upper=3.14159265358979323846 effort=40 velocity=10 -> lower=-3.14159265358979323846 upper=3.14159265358979323846 effort=10 velocity=2
- joint joint6: limit lower=-3.14159265358979323846 upper=3.14159265358979323846 effort=30 velocity=10 -> lower=-3.14159265358979323846 upper=3.14159265358979323846 effort=10 velocity=2
- joint joint7: limit lower=-3.1 upper=3.1 effort=2 velocity=10 -> lower=-3.14159265358979323846 upper=3.14159265358979323846 effort=40 velocity=2; origin xyz=1 0 0 rpy=0 0 0 -> xyz=1 0 0 rpy=1.57079632679489661923 0 0
