Commit message: Bugfixing

File: model/test_4dof.urdf (robot description, URDF)
Before this commit: robot lbr_iiwa, 6 links, 5 joints
Joints:
- joint joint3: limit lower=-3.14159265358979323846 upper=3.14159265358979323846 effort=40 velocity=10 -> lower=-3.14159265358979323846 upper=3.14159265358979323846 effort=60 velocity=10
- joint joint5: limit lower=-3.14159265358979323846 upper=3.14159265358979323846 effort=40 velocity=10 -> lower=-3.1 upper=3.1 effort=2 velocity=10

Commit message: More plotting

File: model/test_4dof.urdf (robot description, URDF)
Before this commit: robot lbr_iiwa, 6 links, 5 joints
Links:
- link world: geometry visual box size=1 0.15 0.15
