Commit message: Bugfixing

File: model/test_2dof.urdf (robot description, URDF)
Before this commit: robot lbr_iiwa, 4 links, 3 joints
Joints:
- joint joint3: limit lower=-3.14159265358979323846 upper=3.14159265358979323846 effort=40 velocity=10 -> lower=-3.14159265358979323846 upper=3.14159265358979323846 effort=60 velocity=10; origin xyz=1 0 0 rpy=1.57079632679489661923 0 0 -> xyz=1 0 0 rpy=0 0 0

File: model/test_4dof.urdf (robot description, URDF)
Before this commit: robot lbr_iiwa, 6 links, 5 joints
Joints:
- joint joint4: limit lower=-3.14159265358979323846 upper=3.14159265358979323846 effort=40 velocity=10 -> lower=-3.14159265358979323846 upper=3.14159265358979323846 effort=40 velocity=5
